Commit message: ROS2 and ros2_control
* Remove separate visualisation package

* Upgrade CMakeLists and package XML to be ament and colcon compatible
for ROS2

* Collapse rviz files into single view_robot file compatible with rviz2

* Rewrite launch file for visualisation

* Restructure urdf files to use a macro for greater potential
extensibility in future (for example, to support hardware versions)

* Add prefix and connected_to arguments

* Add ros2_control data

File: mecademic_description/urdf/meca_500_r3.urdf.xacro (robot description, xacro)
@@ -1,149 +1,23 @@
-<robot name="meca_500_r3" xmlns:xacro="http://ros.org/wiki/xacro">
-  <!-- Base link is the center of the robot's bottom plate -->
-  <link name="meca_base_link">
-    <visual>
-      <origin xyz="0 0 0" rpy="0 0 0" />
-      <geometry>
-        <mesh filename="package://mecademic_description/meshes/meca_500_r3_base.dae" />
-      </geometry>
-    </visual>
-    <collision>
-      <origin xyz="0 0 0" rpy="0 0 0" />
-      <geometry>
-        <mesh filename="package://mecademic_description/meshes/meca_500_r3_base_collision.stl" />
-      </geometry>
-    </collision>
-  </link>
-  <!-- Joint 1 -->
-  <link name="meca_axis_1_link">
-    <visual>
-      <origin xyz="0 0 0" rpy="0 0 0" />
-      <geometry>
-        <mesh filename="package://mecademic_description/meshes/meca_500_r3_j1.dae" />
-      </geometry>
-    </visual>
-    <collision>
-      <origin xyz="0 0 0" rpy="0 0 0" />
-      <geometry>
-        <mesh filename="package://mecademic_description/meshes/meca_500_r3_j1_collision.stl" />
-      </geometry>
-    </collision>
-  </link>
-  <joint name="meca_axis_1_joint" type="revolute">
-    <origin xyz="0.012498 0 0.091" rpy="0 0 0" />
-    <parent link="meca_base_link" />
-    <child link="meca_axis_1_link" />
-    <axis xyz="0 0 1" />
-    <limit effort="10.0" velocity="2.61799" lower="-3.05433" upper="3.05433" />
-  </joint>
-  <!-- Joint 2 -->
-  <link name="meca_axis_2_link">
-    <visual>
-      <origin xyz="0 0 0" rpy="0 0 0" />
-      <geometry>
-        <mesh filename="package://mecademic_description/meshes/meca_500_r3_j2.dae" />
-      </geometry>
-    </visual>
-    <collision>
-      <origin xyz="0 0 0" rpy="0 0 0" />
-      <geometry>
-        <mesh filename="package://mecademic_description/meshes/meca_500_r3_j2_collision.stl" />
-      </geometry>
-    </collision>
-  </link>
-  <joint name="meca_axis_2_joint" type="revolute">
-    <origin xyz="0 0 0.044" rpy="0 0 0" />
-    <parent link="meca_axis_1_link" />
-    <child link="meca_axis_2_link" />
-    <axis xyz="0 1 0" />
-    <limit effort="10.0" velocity="2.61799" lower="-1.22173048" upper="1.5708" />
-  </joint>
-  <!-- Joint 3 -->
-  <link name="meca_axis_3_link">
-    <visual>
-      <origin xyz="0 0 0" rpy="0 0 0" />
-      <geometry>
-        <mesh filename="package://mecademic_description/meshes/meca_500_r3_j3.dae" />
-      </geometry>
-    </visual>
-    <collision>
-      <origin xyz="0 0 0" rpy="0 0 0" />
-      <geometry>
-        <mesh filename="package://mecademic_description/meshes/meca_500_r3_j3_collision.stl" />
-      </geometry>
-    </collision>
-  </link>
-  <joint name="meca_axis_3_joint" type="revolute">
-    <origin xyz="0 0 0.135" rpy="0 0 0" />
-    <parent link="meca_axis_2_link" />
-    <child link="meca_axis_3_link" />
-    <axis xyz="0 1 0" />
-    <limit effort="10.0" velocity="3.14159" lower="-2.35619" upper="1.22173048" />
-  </joint>
-  <!-- Joint 4 -->
-  <link name="meca_axis_4_link">
-    <visual>
-      <origin xyz="0 0 0" rpy="0 0 0" />
-      <geometry>
-        <mesh filename="package://mecademic_description/meshes/meca_500_r3_j4.dae" />
-      </geometry>
-    </visual>
-    <collision>
-      <origin xyz="0 0 0" rpy="0 0 0" />
-      <geometry>
-        <mesh filename="package://mecademic_description/meshes/meca_500_r3_j4_collision.stl" />
-      </geometry>
-    </collision>
-  </link>
-  <joint name="meca_axis_4_joint" type="revolute">
-    <origin xyz="0 0 0.038" rpy="0 0 0" />
-    <parent link="meca_axis_3_link" />
-    <child link="meca_axis_4_link" />
-    <axis xyz="1 0 0" />
-    <limit effort="10.0" velocity="5.23599" lower="-2.96706" upper="2.96706" />
-  </joint>
-  <!-- Joint 5 -->
-  <link name="meca_axis_5_link">
-    <visual>
-      <origin xyz="0 0 0" rpy="0 0 0" />
-      <geometry>
-        <mesh filename="package://mecademic_description/meshes/meca_500_r3_j5.dae" />
-      </geometry>
-    </visual>
-    <collision>
-      <origin xyz="0 0 0" rpy="0 0 0" />
-      <geometry>
-        <mesh filename="package://mecademic_description/meshes/meca_500_r3_j5_collision.stl" />
-      </geometry>
-    </collision>
-  </link>
-  <joint name="meca_axis_5_joint" type="revolute">
-    <origin xyz="0.12 0 0" rpy="0 0 0" />
-    <parent link="meca_axis_4_link" />
-    <child link="meca_axis_5_link" />
-    <axis xyz="0 1 0" />
-    <limit effort="10.0" velocity="5.23599" lower="-2.00713" upper="2.00713" />
-  </joint>
-  <!-- Joint 6 -->
-  <link name="meca_axis_6_link">
-    <visual>
-      <origin xyz="0 0 0" rpy="0 0 0" />
-      <geometry>
-        <mesh filename="package://mecademic_description/meshes/meca_500_r3_j6.dae" />
-      </geometry>
-    </visual>
-    <collision>
-      <origin xyz="0 0 0" rpy="0 0 0" />
-      <geometry>
-        <mesh filename="package://mecademic_description/meshes/meca_500_r3_j6_collision.stl" />
-      </geometry>
-    </collision>
-  </link>
-  <joint name="meca_axis_6_joint" type="revolute">
-    <origin xyz="0.07 0 0" rpy="0 0 0" />
-    <parent link="meca_axis_5_link" />
-    <child link="meca_axis_6_link" />
-    <axis xyz="1 0 0" />
-    <limit effort="10.0" velocity="8.72665" lower="-3.14159" upper="3.14159" />
-  </joint>
+<?xml version="1.0"?>
+<robot xmlns:xacro="http://wiki.ros.org/xacro" name="$(arg name)">
+  <!-- robot name parameter -->
+  <xacro:arg name="name" default="meca_500_r3"/>
+  <!-- import main macro -->
+  <xacro:include filename="$(find mecademic_description)/urdf/meca_500_r3_macro.xacro"/>
+  <!-- parameters -->
+  <xacro:arg name="prefix" default="meca_" />
+  <xacro:arg name="robot_ip" default="" />
+  <xacro:arg name="connected_to" default="" />
+  <xacro:arg name="acceleration_limit" default="30.0" />
+  <!-- ros2_control related parameters -->
+  <xacro:arg name="use_fake_hardware" default="false" />
+  <xacro:arg name="fake_sensor_commands" default="false" />
+  <!-- arm -->
+  <xacro:meca_500_r3_robot
+    prefix="$(arg prefix)"
+    robot_ip="$(arg robot_ip)"
+    connected_to="$(arg connected_to)"
+    acceleration_limit="$(arg acceleration_limit)"
+    use_fake_hardware="$(arg use_fake_hardware)"
+    fake_sensor_commands="$(arg fake_sensor_commands)"/>
 </robot>

Commit message: Support ros2 control (#1)
* ROS2 and ros2_control

* Remove separate visualisation package

* Upgrade CMakeLists and package XML to be ament and colcon compatible
for ROS2

* Collapse rviz files into single view_robot file compatible with rviz2

* Rewrite launch file for visualisation

* Restructure urdf files to use a macro for greater potential
extensibility in future (for example, to support hardware versions)

* Add prefix and connected_to arguments

* Add ros2_control data

* Add port arguments

* Add control and monitoring ports

* Add default values for IP and ports

* Add limit parameters

* Add a velocity timeout parameter that controls the duration in seconds
that a velocity command remains active before the robot automatically
decelerates to a full stop.

* Update acceleration limit to reflect the mecadamic API to be in
percentage units of maximum

* Add velocity limit parameter as a percentage of maximum

* Fix parameter typo

* Remove := from port parameters

* Add missing name argument to launch file

* Add parameter to toggle ros2_control

* Parameter load_ros2_control enables or disables the inclusion
of ros2_control elements in the urdf generation

* meca_500_r3_macro.xacro renamed to just meca_500_r3.xacro

File: mecademic_description/urdf/meca_500_r3.urdf.xacro (robot description, xacro)
@@ -1,149 +1,33 @@
-<robot name="meca_500_r3" xmlns:xacro="http://ros.org/wiki/xacro">
-  <!-- Base link is the center of the robot's bottom plate -->
-  <link name="meca_base_link">
-    <visual>
-      <origin xyz="0 0 0" rpy="0 0 0" />
-      <geometry>
-        <mesh filename="package://mecademic_description/meshes/meca_500_r3_base.dae" />
-      </geometry>
-    </visual>
-    <collision>
-      <origin xyz="0 0 0" rpy="0 0 0" />
-      <geometry>
-        <mesh filename="package://mecademic_description/meshes/meca_500_r3_base_collision.stl" />
-      </geometry>
-    </collision>
-  </link>
-  <!-- Joint 1 -->
-  <link name="meca_axis_1_link">
-    <visual>
-      <origin xyz="0 0 0" rpy="0 0 0" />
-      <geometry>
-        <mesh filename="package://mecademic_description/meshes/meca_500_r3_j1.dae" />
-      </geometry>
-    </visual>
-    <collision>
-      <origin xyz="0 0 0" rpy="0 0 0" />
-      <geometry>
-        <mesh filename="package://mecademic_description/meshes/meca_500_r3_j1_collision.stl" />
-      </geometry>
-    </collision>
-  </link>
-  <joint name="meca_axis_1_joint" type="revolute">
-    <origin xyz="0.012498 0 0.091" rpy="0 0 0" />
-    <parent link="meca_base_link" />
-    <child link="meca_axis_1_link" />
-    <axis xyz="0 0 1" />
-    <limit effort="10.0" velocity="2.61799" lower="-3.05433" upper="3.05433" />
-  </joint>
-  <!-- Joint 2 -->
-  <link name="meca_axis_2_link">
-    <visual>
-      <origin xyz="0 0 0" rpy="0 0 0" />
-      <geometry>
-        <mesh filename="package://mecademic_description/meshes/meca_500_r3_j2.dae" />
-      </geometry>
-    </visual>
-    <collision>
-      <origin xyz="0 0 0" rpy="0 0 0" />
-      <geometry>
-        <mesh filename="package://mecademic_description/meshes/meca_500_r3_j2_collision.stl" />
-      </geometry>
-    </collision>
-  </link>
-  <joint name="meca_axis_2_joint" type="revolute">
-    <origin xyz="0 0 0.044" rpy="0 0 0" />
-    <parent link="meca_axis_1_link" />
-    <child link="meca_axis_2_link" />
-    <axis xyz="0 1 0" />
-    <limit effort="10.0" velocity="2.61799" lower="-1.22173048" upper="1.5708" />
-  </joint>
-  <!-- Joint 3 -->
-  <link name="meca_axis_3_link">
-    <visual>
-      <origin xyz="0 0 0" rpy="0 0 0" />
-      <geometry>
-        <mesh filename="package://mecademic_description/meshes/meca_500_r3_j3.dae" />
-      </geometry>
-    </visual>
-    <collision>
-      <origin xyz="0 0 0" rpy="0 0 0" />
-      <geometry>
-        <mesh filename="package://mecademic_description/meshes/meca_500_r3_j3_collision.stl" />
-      </geometry>
-    </collision>
-  </link>
-  <joint name="meca_axis_3_joint" type="revolute">
-    <origin xyz="0 0 0.135" rpy="0 0 0" />
-    <parent link="meca_axis_2_link" />
-    <child link="meca_axis_3_link" />
-    <axis xyz="0 1 0" />
-    <limit effort="10.0" velocity="3.14159" lower="-2.35619" upper="1.22173048" />
-  </joint>
-  <!-- Joint 4 -->
-  <link name="meca_axis_4_link">
-    <visual>
-      <origin xyz="0 0 0" rpy="0 0 0" />
-      <geometry>
-        <mesh filename="package://mecademic_description/meshes/meca_500_r3_j4.dae" />
-      </geometry>
-    </visual>
-    <collision>
-      <origin xyz="0 0 0" rpy="0 0 0" />
-      <geometry>
-        <mesh filename="package://mecademic_description/meshes/meca_500_r3_j4_collision.stl" />
-      </geometry>
-    </collision>
-  </link>
-  <joint name="meca_axis_4_joint" type="revolute">
-    <origin xyz="0 0 0.038" rpy="0 0 0" />
-    <parent link="meca_axis_3_link" />
-    <child link="meca_axis_4_link" />
-    <axis xyz="1 0 0" />
-    <limit effort="10.0" velocity="5.23599" lower="-2.96706" upper="2.96706" />
-  </joint>
-  <!-- Joint 5 -->
-  <link name="meca_axis_5_link">
-    <visual>
-      <origin xyz="0 0 0" rpy="0 0 0" />
-      <geometry>
-        <mesh filename="package://mecademic_description/meshes/meca_500_r3_j5.dae" />
-      </geometry>
-    </visual>
-    <collision>
-      <origin xyz="0 0 0" rpy="0 0 0" />
-      <geometry>
-        <mesh filename="package://mecademic_description/meshes/meca_500_r3_j5_collision.stl" />
-      </geometry>
-    </collision>
-  </link>
-  <joint name="meca_axis_5_joint" type="revolute">
-    <origin xyz="0.12 0 0" rpy="0 0 0" />
-    <parent link="meca_axis_4_link" />
-    <child link="meca_axis_5_link" />
-    <axis xyz="0 1 0" />
-    <limit effort="10.0" velocity="5.23599" lower="-2.00713" upper="2.00713" />
-  </joint>
-  <!-- Joint 6 -->
-  <link name="meca_axis_6_link">
-    <visual>
-      <origin xyz="0 0 0" rpy="0 0 0" />
-      <geometry>
-        <mesh filename="package://mecademic_description/meshes/meca_500_r3_j6.dae" />
-      </geometry>
-    </visual>
-    <collision>
-      <origin xyz="0 0 0" rpy="0 0 0" />
-      <geometry>
-        <mesh filename="package://mecademic_description/meshes/meca_500_r3_j6_collision.stl" />
-      </geometry>
-    </collision>
-  </link>
-  <joint name="meca_axis_6_joint" type="revolute">
-    <origin xyz="0.07 0 0" rpy="0 0 0" />
-    <parent link="meca_axis_5_link" />
-    <child link="meca_axis_6_link" />
-    <axis xyz="1 0 0" />
-    <limit effort="10.0" velocity="8.72665" lower="-3.14159" upper="3.14159" />
-  </joint>
+<?xml version="1.0"?>
+<robot xmlns:xacro="http://wiki.ros.org/xacro" name="$(arg name)">
+  <!-- robot name parameter -->
+  <xacro:arg name="name" default="meca_500_r3"/>
+  <!-- import main macro -->
+  <xacro:include filename="$(find mecademic_description)/urdf/meca_500_r3.xacro"/>
+  <!-- parameters -->
+  <xacro:arg name="prefix" default="meca_" />
+  <xacro:arg name="robot_ip" default="192.168.0.100" />
+  <xacro:arg name="control_port" default="10000" />
+  <xacro:arg name="monitoring_port" default="10001" />
+  <xacro:arg name="connected_to" default="" />
+  <xacro:arg name="velocity_timeout" default="0.1" />
+  <xacro:arg name="velocity_limit_percent" default="25.0" />
+  <xacro:arg name="acceleration_limit_percent" default="100.0" />
+  <!-- ros2_control related parameters -->
+  <xacro:arg name="load_ros2_control" default="true"/>
+  <xacro:arg name="use_fake_hardware" default="false" />
+  <xacro:arg name="fake_sensor_commands" default="false" />
+  <!-- arm -->
+  <xacro:meca_500_r3_robot
+    prefix="$(arg prefix)"
+    robot_ip="$(arg robot_ip)"
+    control_port="$(arg control_port)"
+    monitoring_port="$(arg monitoring_port)"
+    connected_to="$(arg connected_to)"
+    velocity_timeout="$(arg velocity_timeout)"
+    velocity_limit_percent="$(arg velocity_limit_percent)"
+    acceleration_limit_percent="$(arg acceleration_limit_percent)"
+    load_ros2_control="$(arg load_ros2_control)"
+    use_fake_hardware="$(arg use_fake_hardware)"
+    fake_sensor_commands="$(arg fake_sensor_commands)"/>
 </robot>
