Commit message: Move ros2 control macro to directory and rename to tcpip

File: mecademic_description/ros2_control/meca_500_r3_tcpip.ros2_control.xacro (robot description, xacro)
@@ -1,5 +1,5 @@
 <?xml version="1.0"?>
 <robot xmlns:xacro="http://www.ros.org/wiki/xacro">
-  <xacro:macro name="meca_500_r3_ros2_control" params="
+  <xacro:macro name="meca_500_r3_tcpip_interface" params="
     name
     prefix
@@ -9,24 +9,14 @@
     velocity_timeout
     velocity_limit_percent
-    acceleration_limit_percent
-    use_fake_hardware:=false
-    fake_sensor_commands:=false
-    initial_positions:=${dict(axis_1_joint=0.0,axis_2_joint=0.0,axis_3_joint=0.0,axis_4_joint=0.0,axis_5_joint=0.0,axis_6_joint=0.0)}">
-    <ros2_control name="${name}" type="system">
+    acceleration_limit_percent">
+    <ros2_control name="meca_500_r3_tcpip_interface" type="system">
       <hardware>
-        <xacro:if value="${use_fake_hardware}">
-          <plugin>fake_components/GenericSystem</plugin>
-          <param name="fake_sensor_commands">${fake_sensor_commands}</param>
-          <param name="state_following_offset">0.0</param>
-        </xacro:if>
-        <xacro:unless value="${use_fake_hardware}">
-          <plugin>robot_interface/mecademic/MecademicInterface</plugin>
-          <param name="robot_ip">${robot_ip}</param>
-          <param name="control_port">${control_port}</param>
-          <param name="monitoring_port">${monitoring_port}</param>
-          <param name="velocity_timeout">${velocity_timeout}</param>
-          <param name="velocity_limit_percent">${velocity_limit_percent}</param>
-          <param name="acceleration_limit_percent">${acceleration_limit_percent}</param>
-        </xacro:unless>
+        <plugin>robot_interface/mecademic/MecademicTcpIpInterface</plugin>
+        <param name="robot_ip">${robot_ip}</param>
+        <param name="control_port">${control_port}</param>
+        <param name="monitoring_port">${monitoring_port}</param>
+        <param name="velocity_timeout">${velocity_timeout}</param>
+        <param name="velocity_limit_percent">${velocity_limit_percent}</param>
+        <param name="acceleration_limit_percent">${acceleration_limit_percent}</param>
       </hardware>
       <joint name="${prefix}axis_1_joint">
@@ -42,5 +32,4 @@
         <state_interface name="velocity"/>
         <state_interface name="effort"/>
-        <param name="initial_position">${initial_positions['axis_1_joint']}</param>  <!-- initial position for the FakeSystem -->
       </joint>
       <joint name="${prefix}axis_2_joint">
@@ -56,5 +45,4 @@
         <state_interface name="velocity"/>
         <state_interface name="effort"/>
-        <param name="initial_position">${initial_positions['axis_2_joint']}</param>  <!-- initial position for the FakeSystem -->
       </joint>
       <joint name="${prefix}axis_3_joint">
@@ -70,5 +58,4 @@
         <state_interface name="velocity"/>
         <state_interface name="effort"/>
-        <param name="initial_position">${initial_positions['axis_3_joint']}</param>  <!-- initial position for the FakeSystem -->
       </joint>
       <joint name="${prefix}axis_4_joint">
@@ -84,5 +71,4 @@
         <state_interface name="velocity"/>
         <state_interface name="effort"/>
-        <param name="initial_position">${initial_positions['axis_4_joint']}</param>  <!-- initial position for the FakeSystem -->
       </joint>
       <joint name="${prefix}axis_5_joint">
@@ -98,5 +84,4 @@
         <state_interface name="velocity"/>
         <state_interface name="effort"/>
-        <param name="initial_position">${initial_positions['axis_5_joint']}</param>  <!-- initial position for the FakeSystem -->
       </joint>
       <joint name="${prefix}axis_6_joint">
@@ -112,5 +97,4 @@
         <state_interface name="velocity"/>
         <state_interface name="effort"/>
-        <param name="initial_position">${initial_positions['axis_6_joint']}</param>  <!-- initial position for the FakeSystem -->
       </joint>
     </ros2_control>

File: mecademic_description/urdf/meca_500_r3.xacro (robot description, xacro)
@@ -1,33 +1,5 @@
 <?xml version="1.0"?>
 <robot xmlns:xacro="http://wiki.ros.org/xacro">
-  <xacro:macro name="meca_500_r3_robot" params="
-    prefix
-    robot_ip
-    control_port
-    monitoring_port
-    connected_to:=''
-    velocity_timeout:=0.1
-    velocity_limit_percent:=25.0
-    acceleration_limit_percent:=100.0
-    load_ros2_control:=true
-    use_fake_hardware:=false
-    fake_sensor_commands:=false
-    initial_positions:=${dict(axis_1_joint=0.0,axis_2_joint=0.0,axis_3_joint=0.0,axis_4_joint=0.0,axis_5_joint=0.0,axis_6_joint=0.0)}">
-    <xacro:if value="${load_ros2_control}">
-      <!-- ros2 control include -->
-      <xacro:include filename="$(find mecademic_description)/urdf/meca_500_r3.ros2_control.xacro" />
-      <!-- ros2 control instance -->
-      <xacro:meca_500_r3_ros2_control
-        name="MecademicInterface"
-        prefix="${prefix}"
-        robot_ip="$(arg robot_ip)"
-        control_port="$(arg control_port)"
-        monitoring_port="$(arg monitoring_port)"
-        velocity_timeout="$(arg velocity_timeout)"
-        velocity_limit_percent="$(arg velocity_limit_percent)"
-        acceleration_limit_percent="$(arg acceleration_limit_percent)"
-        use_fake_hardware="$(arg use_fake_hardware)"
-        fake_sensor_commands="$(arg fake_sensor_commands)"/>
-    </xacro:if>
+  <xacro:macro name="meca_500_r3" params="prefix connected_to:=''">
     <xacro:if value="${connected_to == ''}">
       <link name="world" />

Commit message: Add macros for ethercat interface (#4)
* Remove not needed files

* Move ros2 control macro to directory and rename to tcpip

* Add macros for ecat version

* Update package files

* Fixes

File: mecademic_description/ros2_control/meca_500_r3_tcpip.ros2_control.xacro (robot description, xacro)
@@ -1,6 +1,5 @@
 <?xml version="1.0"?>
 <robot xmlns:xacro="http://www.ros.org/wiki/xacro">
-  <xacro:macro name="meca_500_r3_ros2_control" params="
-    name
+  <xacro:macro name="meca_500_r3_tcpip_interface" params="
     prefix
     robot_ip
@@ -9,24 +8,14 @@
     velocity_timeout
     velocity_limit_percent
-    acceleration_limit_percent
-    use_fake_hardware:=false
-    fake_sensor_commands:=false
-    initial_positions:=${dict(axis_1_joint=0.0,axis_2_joint=0.0,axis_3_joint=0.0,axis_4_joint=0.0,axis_5_joint=0.0,axis_6_joint=0.0)}">
-    <ros2_control name="${name}" type="system">
+    acceleration_limit_percent">
+    <ros2_control name="meca_500_r3_tcpip_interface" type="system">
       <hardware>
-        <xacro:if value="${use_fake_hardware}">
-          <plugin>fake_components/GenericSystem</plugin>
-          <param name="fake_sensor_commands">${fake_sensor_commands}</param>
-          <param name="state_following_offset">0.0</param>
-        </xacro:if>
-        <xacro:unless value="${use_fake_hardware}">
-          <plugin>robot_interface/mecademic/MecademicInterface</plugin>
-          <param name="robot_ip">${robot_ip}</param>
-          <param name="control_port">${control_port}</param>
-          <param name="monitoring_port">${monitoring_port}</param>
-          <param name="velocity_timeout">${velocity_timeout}</param>
-          <param name="velocity_limit_percent">${velocity_limit_percent}</param>
-          <param name="acceleration_limit_percent">${acceleration_limit_percent}</param>
-        </xacro:unless>
+        <plugin>robot_interface/mecademic/MecademicTcpIpInterface</plugin>
+        <param name="robot_ip">${robot_ip}</param>
+        <param name="control_port">${control_port}</param>
+        <param name="monitoring_port">${monitoring_port}</param>
+        <param name="velocity_timeout">${velocity_timeout}</param>
+        <param name="velocity_limit_percent">${velocity_limit_percent}</param>
+        <param name="acceleration_limit_percent">${acceleration_limit_percent}</param>
       </hardware>
       <joint name="${prefix}axis_1_joint">
@@ -42,5 +31,4 @@
         <state_interface name="velocity"/>
         <state_interface name="effort"/>
-        <param name="initial_position">${initial_positions['axis_1_joint']}</param>  <!-- initial position for the FakeSystem -->
       </joint>
       <joint name="${prefix}axis_2_joint">
@@ -56,5 +44,4 @@
         <state_interface name="velocity"/>
         <state_interface name="effort"/>
-        <param name="initial_position">${initial_positions['axis_2_joint']}</param>  <!-- initial position for the FakeSystem -->
       </joint>
       <joint name="${prefix}axis_3_joint">
@@ -70,5 +57,4 @@
         <state_interface name="velocity"/>
         <state_interface name="effort"/>
-        <param name="initial_position">${initial_positions['axis_3_joint']}</param>  <!-- initial position for the FakeSystem -->
       </joint>
       <joint name="${prefix}axis_4_joint">
@@ -84,5 +70,4 @@
         <state_interface name="velocity"/>
         <state_interface name="effort"/>
-        <param name="initial_position">${initial_positions['axis_4_joint']}</param>  <!-- initial position for the FakeSystem -->
       </joint>
       <joint name="${prefix}axis_5_joint">
@@ -98,5 +83,4 @@
         <state_interface name="velocity"/>
         <state_interface name="effort"/>
-        <param name="initial_position">${initial_positions['axis_5_joint']}</param>  <!-- initial position for the FakeSystem -->
       </joint>
       <joint name="${prefix}axis_6_joint">
@@ -112,5 +96,4 @@
         <state_interface name="velocity"/>
         <state_interface name="effort"/>
-        <param name="initial_position">${initial_positions['axis_6_joint']}</param>  <!-- initial position for the FakeSystem -->
       </joint>
     </ros2_control>
